File: Circuits/control_board/Control_board.kicad_sch (KiCad schematic)
At the start: 34 parts, among them J1 Conn_01x01_Female, J2 Conn_01x01_Female, J3 Conn_01x01_Female, J4 Conn_01x01_Female, J5 Conn_01x01_Female, J6 Conn_01x01_Female, Q1 S8050, U1 PC817, U2 PC817, U3 PC817, U4 PC817

Commit message: further development in circuit
Parts:
- added Q2: S8050, Package_TO_SOT_THT:TO-92_Inline, symbol Transistor_BJT:S8050
- added U5: TL062, symbol Amplifier_Operational:TL062
- added U6: LM393, symbol Comparator:LM393
- added U7: TL431LP, Package_TO_SOT_THT:TO-92_Inline, symbol Reference_Voltage:TL431LP
Other:
- moved on the sheet: J1, J2, J3, J4, J5, J6, QN1, QN2, QP1, QP2, R5, R6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

Commit message: Updated control circuitry schematics
Parts:
- removed J1, J2, J3, J4, J5, J6: Conn_01x01_Female, Connector_PinSocket_2.54mm:PinSocket_1x01_P2.54mm_Vertical, symbol Connector:Conn_01x01_Female
- removed R? (x5): 1k, Resistor_THT:R_Axial_DIN0207_L6.3mm_D2.5mm_P7.62mm_Horizontal, symbol Device:R
- added C2, C4: 1uF, symbol Device:C_Polarized
- added C3: C, Capacitor_THT:C_Disc_D5.0mm_W2.5mm_P2.50mm, symbol Device:C
- added D1: LED, symbol Device:LED
- added J1: Pic UART, Connector_PinSocket_2.54mm:PinSocket_1x02_P2.54mm_Vertical, symbol Connector:Conn_01x02_Socket
- added PowerInput: 12v, TerminalBlock:TerminalBlock_bornier-2_P5.08mm, symbol Connector:Screw_Terminal_01x02
- added Q3: S8550, Package_TO_SOT_THT:TO-92_Inline, symbol Transistor_BJT:S8550
- added R1, R11, R9: 220, Resistor_THT:R_Axial_DIN0207_L6.3mm_D2.5mm_P7.62mm_Horizontal, symbol Device:R
- added R10: 5k, Resistor_THT:R_Axial_DIN0207_L6.3mm_D2.5mm_P7.62mm_Horizontal, symbol Device:R
- added R12, R14, R17, R18, R23, R24, R25, R26: 1k, Resistor_THT:R_Axial_DIN0207_L6.3mm_D2.5mm_P7.62mm_Horizontal, symbol Device:R
- added R13, R15: 10k, Resistor_THT:R_Axial_DIN0207_L6.3mm_D2.5mm_P7.62mm_Horizontal, symbol Device:R
- added R16: 470, Resistor_THT:R_Axial_DIN0207_L6.3mm_D2.5mm_P7.62mm_Horizontal, symbol Device:R
- added R19: 330, Resistor_THT:R_Axial_DIN0207_L6.3mm_D2.5mm_P7.62mm_Horizontal, symbol Device:R
- added R20, R21, R22: ?, Resistor_THT:R_Axial_DIN0207_L6.3mm_D2.5mm_P7.62mm_Horizontal, symbol Device:R
- added RV1: 10k, Connector_PinSocket_2.54mm:PinSocket_1x03_P2.54mm_Vertical, symbol Device:R_Potentiometer_Trim
- added RV2: 10K, Connector_PinSocket_2.54mm:PinSocket_1x03_P2.54mm_Vertical, symbol Device:R_Potentiometer_Trim
- added RV3: 1k, Connector_PinSocket_2.54mm:PinSocket_1x03_P2.54mm_Vertical, symbol Device:R_Potentiometer_Trim
- added R_Shunt1, R_Shunt2: 2 ohm, Resistor_THT:R_Axial_Shunt_L22.2mm_W9.5mm_PS14.30mm_P25.40mm, symbol Device:R_Shunt
- added U10: PIC18F2550-ISP, Package_DIP:DIP-28_W7.62mm, symbol MCU_Microchip_PIC18:PIC18F2550-ISP
- added U11, U9: LM317_TO-220, Package_TO_SOT_THT:TO-220-3_Vertical, symbol Regulator_Linear:LM317_TO-220
- added U8: TL062, symbol Amplifier_Operational:TL062
- R0: value 5k -> 1k
Connections:
- net +12V: now also C1.1, R4.1, U5.8 (V+), U6.8 (V+), C3.1, PowerInput.1 (Pin_1), Q3.1 (E), R15.1, R17.2, U11.3 (VI), U9.3 (VI); no longer QP1.2 (E), QP2.2 (E), R5.1, R6.1, R7.1, R8.1
- net +5V: now also C4.1, R21.1, U11.2 (VO); no longer R0.2, R2.2, R4.1
- net GND: now also C1.2, Q2.1 (E), U5.4 (V-), U6.4 (V-), U7.2 (A), C2.2, C3.2, C4.2, D1.1 (K), PowerInput.2 (Pin_2), R10.2, R14.1, R22.2, RV2.3, U8.4 (V-)
- net at U3.1: now also R24.2
- net DC_Motor_P2: now reaches QN2.1 (C), QP2.1 (C)
- net at U4.1: now also R25.1
- net at Q1.2 (B), Q?.3 (C), R0.1: now also R19.1
- net at Q?.2 (B): now also R18.1
- net DC_Motor_P1: now reaches QN1.1 (C), QP1.1 (C)
- net at U6.1: now also Q2.2 (B), R15.2
- net 3.4V REFRENCE: now reaches U6.2 (-)
- net 3.4V REFRENCE: now also U7.3 (K), R12.1, RV3.2
- net at U6.3 (+): now also R13.2
- net V_current: now reaches U5.1
- net V_current: now also R11.2, RV1.2
- net at U5.2 (-): now also R11.1, R9.1
- net at U5.3 (+): now also R1.2, R10.1
- net Thermistor_reading: now reaches R3.2, ThermistorInput.2 (Pin_2)
- net at U2.1: now also R26.1
- net at U1.1: now also R23.2
- net at Q2.3 (C): now also R16.1
- net at U7.1 (REF): now also R14.2
- new net: Q3.3 (C), U8.8 (V+)
- new net: Q3.2 (B), R16.2, R17.1
- new net: D1.2 (A), R19.2
- new net: R21.2, R22.1, U11.1 (ADJ)
- new net G1_pin: R24.1
- new net G2_pin: R25.2
- new net Heater_control_pin: R18.2
- new net V1_pin: R23.1
- new net V2_pin: R26.2
- new net VCC: C2.1, R1.1, R20.1, R_Shunt1.1, R_Shunt2.1, U9.2 (VO)
- new net VS: QP1.2 (E), QP2.2 (E), R5.1, R6.1, R7.1, R8.1, R9.2, R_Shunt1.4, R_Shunt2.4
- new net V_current_divided: R13.1, RV1.3, RV2.2, U8.3 (+)
- new net V_current_divided_clamped: U8.1, U8.2 (-)
Other:
- note added: "**Check the importance of the seperation resistor, I really think it's useless"
- note added: "**Deciding the Power supply of the constant voltage has no practical importance except for when designing the PCB, should choose the easier to route"
- note added: "**Deciding the Power supply of the control transistorhas no practical importance except for when designing the PCB, should choose the easier to route ** Also check these resistor values"
- note added: "**Design the 1-2 Demultiplexer for the G2 motor pin"
- note added: "**Must decide whether pic uC will be powered from the same 3-5v from the linear voltage regulator or will have a stand alone 5v linear voltage regular. This will depend on oscilloscope testing and whether having a seperate linear voltage regulator really removes/reduces dc motor noise"
- note added: "**No MCP4313 chip in kicad library Must design the MCP4313 chip in Kicad"
- note added: "**Rigourisly check if this LED doesn't disturb the PWM signal to the darlington power transistor"
- note added: "**THIS IS THE OLD SCHEMATIC OF THE H-BRIDGE! MUST UPDATE!!!"
- note added: "**Think about how to incorporate a TTL converter chip on the PCB"
- note added: "**and how the USB output of the ttl converter will come out of the PCB, a female micro-usb? a female usb-c?"
- note added: "**check the inverting and non-inverting pin"
- note added: "Constant 3.4V Refrence for comparator to compare against VA_Block signal"
- note added: "H-Bridge"
- note added: "Heater Power Control"
- note added: "Over-Voltage Protection: to protect uC from spikes from current readings"
- note added: "The 5v will only be used for the Pic uC, MCP4131 and the digital logic ICs"
- note added: "Thermistor"
- note added: "VA_Block: Measures current"
- note added: "Voltage Divider: to get the Motor maximum current reading in under 3.3v"
- note added: "Will take same Vcc as uC. For micropython boards outside. unfortionately must have to make voltage divider on a breadboard outside the PCB if needed :("
- moved on the sheet: C1, D?, HeaterOutput, Q1, Q2, Q?, QD1, QN1, QN2, QP1, QP2, R0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

Commit message: Further development in circuit schematics and pic code, including demultiplexer circuit
Parts:
- removed D1: LED, symbol Device:LED
- added D2: LED, symbol Device:LED
- added Q4: S8050, Package_TO_SOT_THT:TO-92_Inline, symbol Transistor_BJT:S8050
- added R27: 330, Resistor_THT:R_Axial_DIN0207_L6.3mm_D2.5mm_P7.62mm_Horizontal, symbol Device:R
- added U12: MCP41010, symbol Potentiometer_Digital:MCP41010
- added U13: 7400, symbol 74xx:7400
- J1: value Pic UART -> Pic UART JST Connector; footprint Connector_PinSocket_2.54mm:PinSocket_1x02_P2.54mm_Vertical -> Connector_PinSocket_2.54mm:PinSocket_1x02_P2.54mm_Horizontal
- R19: value 330 -> 4.7k
- R20: value ? -> 2.2k
- R21: value ? -> 3.3k
- R22: value ? -> 1.2k
Connections:
- net +5V: now also R19.2, U12.8 (VDD), U13.14 (VCC)
- net G1_pin: now also U13.3
- net G2_pin: now also U13.6
- net GND: now also Q4.1 (E), U12.4 (VSS), U12.7 (PB0), U13.7 (GND)
- net Heater_control_pin: now also U10.13 (CCP1/RC2)
- net Thermistor_reading: now also U10.2 (RA0/AN0)
- net V1_pin: now also U10.24 (RB3/AN9/CCP2/VPO)
- net V2_pin: now also U10.25 (RB4/AN11/KBI0)
- net V_current_divided_clamped: now also U10.3 (RA1/AN1)
- net at Q1.2 (B), Q?.3 (C), R0.1: now also R27.1; no longer R19.1
- net UART_TX_Pin: now reaches J1.1 (Pin_1)
- net UART_TX_Pin: now also U10.17 (TX/CK/RC6)
- net UART_RX_Pin: now reaches J1.2 (Pin_2)
- net UART_RX_Pin: now also U10.18 (SDO/RX/DT/RC7)
- net at U9.1 (ADJ): now also R20.2, U12.6 (PW0)
- net MCP_CS_Pin: now reaches U10.11 (T1OSO/T13CKI/RC0)
- net MCP_CS_Pin: now also U12.1 (~{CS})
- net Demultiplexer_Input_Signal: now reaches U10.12 (~{UOE}/CCP2/T1OSI/RC1)
- net Demultiplexer_Input_Signal: now also U13.2, U13.5
- net SDI_Pin: now reaches U10.21 (RB0/AN12/INT0/FLT0/SDI/SDA)
- net SDI_Pin: now also U12.3 (SI/SO)
- net SCK_Pin: now reaches U10.22 (RB1/AN10/INT1/SCK/SCL)
- net SCK_Pin: now also U12.2 (SCK)
- net Demultiplexer Select Pin: now reaches U10.26 (RB5/KBI1/PGM)
- net Demultiplexer Select Pin: now also Q4.2 (B), U13.1
- new net: D2.2 (A), R27.2
- new net: Q4.3 (C), R19.1, U13.4
Other:
- note added: "** I think I need to design a multiplexer to control when SDI/SDO enters the IC"
- note added: "** decide to connect to which Pic GND pin when designing PCB"
- note added: "** test if it's really okay to connect UART RX and SPI SDO to the same pin"
- note added: "Demultiplexer: to demultiplexer the PWM signal to the wanted Motor GND Pin, the one with wanted CW/CCW"
- note added: "Main Pic Controller"
- note added: "The 5v will only be used for the Pic uC, MCP4131 and the demultiplexer logic circuitry"
- note removed: "**Must decide whether pic uC will be powered from the same 3-5v from the linear voltage regulator or will have a stand alone 5v linear voltage regular. This will depend on oscilloscope testing and whether having a seperate linear voltage regulator really removes/reduces dc motor noise"
- note removed: "**No MCP4313 chip in kicad library Must design the MCP4313 chip in Kicad"
- note removed: "**Think about how to incorporate a TTL converter chip on the PCB"
- note removed: "**and how the USB output of the ttl converter will come out of the PCB, a female micro-usb? a female usb-c?"
- note removed: "The 5v will only be used for the Pic uC, MCP4131 and the digital logic ICs"
- moved on the sheet: C1, C2, J1, PowerInput, R20, U10, U9

Commit message: minor changes to circuit
Parts:
- removed R21: 3.3k, Resistor_THT:R_Axial_DIN0207_L6.3mm_D2.5mm_P7.62mm_Horizontal, symbol Device:R
- removed R22: 1.2k, Resistor_THT:R_Axial_DIN0207_L6.3mm_D2.5mm_P7.62mm_Horizontal, symbol Device:R
- removed U11: LM317_TO-220, Package_TO_SOT_THT:TO-220-3_Vertical, symbol Regulator_Linear:LM317_TO-220
- added U14: L7805, symbol Regulator_Linear:L7805
Connections:
- net +12V: now also U14.1 (IN)
- net +5V: now also U14.3 (OUT)
- net GND: now also U14.2 (GND)
Changed lines of the file:
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@@
   (junction (at 406.4 138.43) (diameter 0) (color 0 0 0 0)
   )
-  (junction (at 81.28 -39.37) (diameter 0) (color 0 0 0 0)
-  )
   (junction (at 139.7 -62.23) (diameter 0) (color 0 0 0 0)
   )
@@
   (junction (at 132.08 46.99) (diameter 0) (color 0 0 0 0)
   )
-  (junction (at 72.39 -12.7) (diameter 0) (color 0 0 0 0)
+  (junction (at 72.39 -21.59) (diameter 0) (color 0 0 0 0)
   )
   (junction (at 68.58 127) (diameter 0) (color 0 0 0 0)
@@
   (junction (at 270.51 123.19) (diameter 0) (color 0 0 0 0)
   )
-  (junction (at 72.39 -26.67) (diameter 0) (color 0 0 0 0)
-  )
   (junction (at -127 107.95) (diameter 0) (color 0 0 0 0)
   )
@@
     (stroke (width 0) (type default))
   )
+  (wire (pts (xy 55.88 -26.67) (xy 55.88 -21.59))
+    (stroke (width 0) (type default))
+  )
   (wire (pts (xy 226.06 43.18) (xy 248.92 43.18))
     (stroke (width 0) (type default))
@@
     (stroke (width 0) (type default))
   )
-  (wire (pts (xy 90.17 -12.7) (xy 90.17 -26.67))
-    (stroke (width 0) (type default))
-  )
   (wire (pts (xy 119.38 148.59) (xy 119.38 154.94))
     (stroke (width 0) (type default))
@@
     (stroke (width 0) (type default))
   )
-  (wire (pts (xy 55.88 -26.67) (xy 55.88 -12.7))
+  (wire (pts (xy 72.39 -31.75) (xy 72.39 -21.59))
     (stroke (width 0) (type default))
   )
@@
     (stroke (width 0) (type default))
   )
-  (wire (pts (xy 81.28 -39.37) (xy 80.01 -39.37))
+  (wire (pts (xy 80.01 -39.37) (xy 90.17 -39.37))
     (stroke (width 0) (type default))
   )
@@
     (stroke (width 0) (type default))
   )
-  (wire (pts (xy 72.39 -31.75) (xy 72.39 -26.67))
-    (stroke (width 0) (type default))
-  )
   (wire (pts (xy 157.48 54.61) (xy 160.02 54.61))
     (stroke (width 0) (type default))
@@
     (stroke (width 0) (type default))
   )
-  (wire (pts (xy 81.28 -39.37) (xy 81.28 -34.29))
-    (stroke (width 0) (type default))
-  )
   (wire (pts (xy 124.46 57.15) (xy 124.46 72.39))
     (stroke (width 0) (type default))
@@
     (stroke (width 0) (type default))
   )
-  (wire (pts (xy 90.17 -39.37) (xy 81.28 -39.37))
-    (stroke (width 0) (type default))
-  )
   (wire (pts (xy 66.04 134.62) (xy 66.04 140.97))
     (stroke (width 0) (type default))
@@
     (stroke (width 0) (type default))
   )
-  (wire (pts (xy 55.88 -12.7) (xy 72.39 -12.7))
-    (stroke (width 0) (type default))
-  )
-  (wire (pts (xy 72.39 -26.67) (xy 72.39 -24.13))
+  (wire (pts (xy 55.88 -21.59) (xy 72.39 -21.59))
     (stroke (width 0) (type default))
   )
@@
     (stroke (width 0) (type default))
   )
-  (wire (pts (xy 72.39 -26.67) (xy 81.28 -26.67))
-    (stroke (width 0) (type default))
-  )
   (wire (pts (xy 191.77 -71.12) (xy 191.77 -66.04))
     (stroke (width 0) (type default))
@@
     (stroke (width 0) (type default))
   )
-  (wire (pts (xy 72.39 -16.51) (xy 72.39 -12.7))
-    (stroke (width 0) (type default))
-  )
   (wire (pts (xy 248.92 43.18) (xy 248.92 50.8))
     (stroke (width 0) (type default))
@@
     (stroke (width 0) (type default))
   )
+  (wire (pts (xy 90.17 -26.67) (xy 90.17 -21.59))
+    (stroke (width 0) (type default))
+  )
   (wire (pts (xy 388.62 115.57) (xy 427.99 115.57))
     (stroke (width 0) (type default))
@@
     (stroke (width 0) (type default))
   )
-  (wire (pts (xy 72.39 -12.7) (xy 90.17 -12.7))
+  (wire (pts (xy 72.39 -21.59) (xy 90.17 -21.59))
     (stroke (width 0) (type default))
   )
@@
     )
   )
-  (symbol (lib_id "power:GND") (at 72.39 -12.7 0) (unit 1)
+  (symbol (lib_id "power:GND") (at 72.39 -21.59 0) (unit 1)
     (in_bom yes) (on_board yes) (dnp no) (fields_autoplaced)
-    (property "Reference" "#PWR024" (at 72.39 -6.35 0)
+    (property "Reference" "#PWR024" (at 72.39 -15.24 0)
       (effects (font (size 1.27 1.27)) hide)
     )
-    (property "Value" "GND" (at 72.39 -8.2566 0)
+    (property "Value" "GND" (at 72.39 -17.1466 0)
       (effects (font (size 1.27 1.27)))
     )
-    (property "Footprint" "" (at 72.39 -12.7 0)
+    (property "Footprint" "" (at 72.39 -21.59 0)
       (effects (font (size 1.27 1.27)) hide)
     )
-    (property "Datasheet" "" (at 72.39 -12.7 0)
+    (property "Datasheet" "" (at 72.39 -21.59 0)
       (effects (font (size 1.27 1.27)) hide)
     )
@@
     )
   )
-  (symbol (lib_id "Regulator_Linear:LM317_TO-220") (at 72.39 -39.37 0) (unit 1)
-    (in_bom yes) (on_board yes) (dnp no) (fields_autoplaced)
-    (property "Reference" "U11" (at 72.39 -44.45 0)
-      (effects (font (size 1.27 1.27)))
-    )
-    (property "Value" "LM317_TO-220" (at 72.39 -41.91 0)
-      (effects (font (size 1.27 1.27)))
-    )
-    (property "Footprint" "Package_TO_SOT_THT:TO-220-3_Vertical" (at 72.39 -45.72 0)
-      (effects (font (size 1.27 1.27) italic) hide)
-    )
-    (property "Datasheet" "http://www.ti.com/lit/ds/symlink/lm317.pdf" (at 72.39 -39.37 0)
-      (effects (font (size 1.27 1.27)) hide)
-    )
-    (pin "1")
-    (pin "2")
-    (pin "3")
-    (instances
-      (project "Control_board"
-        (path "/e63e39d7-6ac0-4ffd-8aa3-1841a4541b55"
-          (reference "U11") (unit 1)
-        )
-      )
-    )
-  )
   (symbol (lib_id "Device:R") (at 111.76 -34.29 0) (unit 1)
     (in_bom yes) (on_board yes) (dnp no) (fields_autoplaced)
@@
     )
   )
-  (symbol (lib_id "Device:R") (at 72.39 -20.32 0) (unit 1)
-    (in_bom yes) (on_board yes) (dnp no) (fields_autoplaced)
-    (property "Reference" "R22" (at 74.168 -21.1547 0)
-      (effects (font (size 1.27 1.27)) (justify left))
-    )
-    (property "Value" "1.2k" (at 74.168 -18.6178 0)
-      (effects (font (size 1.27 1.27)) (justify left))
-    )
-    (property "Footprint" "Resistor_THT:R_Axial_DIN0207_L6.3mm_D2.5mm_P7.62mm_Horizontal" (at 70.612 -20.32 90)
-      (effects (font (size 1.27 1.27)) hide)
-    )
-    (property "Datasheet" "~" (at 72.39 -20.32 0)
-      (effects (font (size 1.27 1.27)) hide)
-    )
-    (pin "1")
-    (pin "2")
-    (instances
-      (project "Control_board"
-        (path "/e63e39d7-6ac0-4ffd-8aa3-1841a4541b55"
-          (reference "R22") (unit 1)
-        )
-      )
-    )
-  )
   (symbol (lib_id "power:+5V") (at -127 95.25 0) (unit 1)
     (in_bom yes) (on_board yes) (dnp no) (fields_autoplaced)
@@
     )
   )
-  (symbol (lib_id "Device:R") (at 81.28 -30.48 0) (unit 1)
-    (in_bom yes) (on_board yes) (dnp no) (fields_autoplaced)
-    (property "Reference" "R21" (at 83.058 -31.3147 0)
-      (effects (font (size 1.27 1.27)) (justify left))
-    )
-    (property "Value" "3.3k" (at 83.058 -28.7778 0)
-      (effects (font (size 1.27 1.27)) (justify left))
-    )
-    (property "Footprint" "Resistor_THT:R_Axial_DIN0207_L6.3mm_D2.5mm_P7.62mm_Horizontal" (at 79.502 -30.48 90)
-      (effects (font (size 1.27 1.27)) hide)
-    )
-    (property "Datasheet" "~" (at 81.28 -30.48 0)
-      (effects (font (size 1.27 1.27)) hide)
-    )
-    (pin "1")
-    (pin "2")
-    (instances
-      (project "Control_board"
-        (path "/e63e39d7-6ac0-4ffd-8aa3-1841a4541b55"
-          (reference "R21") (unit 1)
-        )
-      )
-    )
-  )
   (symbol (lib_id "Device:R") (at -55.88 109.22 180) (unit 1)
     (in_bom yes) (on_board yes) (dnp no) (fields_autoplaced)
@@
         )
       )
+    )
+  )
+  (symbol (lib_id "Regulator_Linear:L7805") (at 72.39 -39.37 0) (unit 1)
+    (in_bom yes) (on_board yes) (dnp no) (fields_autoplaced)
+    (property "Reference" "U14" (at 72.39 -44.45 0)
+      (effects (font (size 1.27 1.27)))
+    )
+    (property "Value" "L7805" (at 72.39 -41.91 0)
+      (effects (font (size 1.27 1.27)))
+    )
+    (property "Footprint" "" (at 73.025 -35.56 0)
+      (effects (font (size 1.27 1.27) italic) (justify left) hide)
+    )
+    (property "Datasheet" "http://www.st.com/content/ccc/resource/technical/document/datasheet/41/4f/b3/b0/12/d4/47/88/CD00000444.pdf/files/CD00000444.pdf/jcr:content/translations/en.CD00000444.pdf" (at 72.39 -38.1 0)
+      (effects (font (size 1.27 1.27)) hide)
+    )
+    (pin "1")
+    (pin "2")
+    (pin "3")
+    (instances
+      (project "Control_board"
+        (path "/e63e39d7-6ac0-4ffd-8aa3-1841a4541b55"
+          (reference "U14") (unit 1)
+        )
+      )

Commit message: removed the MCP4131 digital potentiometer idea as it can only handle 7v
Parts:
- removed U12: MCP41010, symbol Potentiometer_Digital:MCP41010
- added C5, C6, C7: 0.1uF, Capacitor_THT:C_Disc_D5.0mm_W2.5mm_P2.50mm, symbol Device:C
- added RV4: 10k, symbol Device:R_Potentiometer_Trim
- added Y1: Crystal, symbol Device:Crystal
- C3: value C -> 0.1uF
Connections:
- net +12V: now also C5.1, C6.1
- net GND: now also C5.2, C6.2, C7.1, RV4.2
- net at Q3.3 (C), U8.8 (V+): now also C7.2
- net at R20.2, U9.1 (ADJ): now also RV4.1
- net at U10.10 (RA6/OSC2/CLKO): now also Y1.2
- net at U10.9 (OSC1/CLKI): now also Y1.1
- net SCK_Pin: no longer names the net of U10.22 (RB1/AN10/INT1/SCK/SCL)
- net SDI_Pin: no longer names the net of U10.21 (RB0/AN12/INT0/FLT0/SDI/SDA)
Other:
- note added: "**Decide on what potentiometer to use here"
- note removed: "** I think I need to design a multiplexer to control when SDI/SDO enters the IC"
